File: Cinema Display/Cinema Display Barrel Jack Adapter/Cinema Display Barrel Jack Adapter.kicad_pcb (KiCad board)
At the start: 2 copper layers, 16 x 25 mm, 3 parts, among them J1 CINEMA-DISPLAY-POWER-CONNECTOR, J2 54-00253

Commit message: Added copyright information.
Other:
- board text added: "The Electron Vault"
- board text added: "©2026"
Changed lines of the file:
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@@
 		(descr "Tensility 54-00253")
 		(property "Reference" "J2"
-			(at 6.5 -7.5 0)
+			(at -5 -7.5 0)
 			(layer "F.SilkS")
 			(effects
@@
 		)
 		(property "Value" "54-00253"
-			(at 0 6.999999 360)
+			(at 0 6.999999 0)
 			(layer "F.Fab")
 			(effects
@@
 		)
 		(property "Footprint" "Cinema Display Barrel Jack Adapter_Footprints:54-00253"
-			(at 0 4.800001 360)
+			(at 0 4.800001 0)
 			(layer "F.Fab")
 			(hide yes)
@@
 		)
 		(property "Datasheet" "-"
-			(at 0 4.800001 360)
+			(at 0 4.800001 0)
 			(layer "F.Fab")
 			(hide yes)
@@
 		)
 		(property "Description" "CONN BARREL JACK 2.1 x 5.5mm"
-			(at 0 4.800001 360)
+			(at 0 4.800001 0)
 			(layer "F.Fab")
 			(hide yes)
@@
 		(fp_arc
 			(start -5.1 -5.4)
-			(mid -4.953553 -5.753552)
+			(mid -4.953553 -5.753553)
 			(end -4.6 -5.9)
 			(stroke
@@
 		)
 		(fp_text user "${REFERENCE}"
-			(at 0 0 360)
+			(at 0 0 0)
 			(layer "F.Fab")
 			(effects
@@
 		(layer "Edge.Cuts")
 	)
+	(gr_text "©2026"
+		(at 107.26 120.5 90)
+		(layer "F.SilkS")
+		(effects
+			(font
+				(size 0.9 0.9)
+				(thickness 0.2)
+				(bold yes)
+			)
+			(justify left bottom)
+		)
+	)
+	(gr_text "The Electron Vault"
+		(at 105.56 128.4 90)
+		(layer "F.SilkS")
+		(effects
+			(font
+				(size 0.9 0.9)
+				(thickness 0.2)
+				(bold yes)
+			)
+			(justify left bottom)
+		)
+	)
 	(gr_text "Min track/spacing: "
